File: kicad/YAMS - Yet Another Motion Sensor.kicad_pcb (KiCad board)
At the start: 2 copper layers, 34.3 x 51.4 mm, 12 parts, among them J1 Power, J2 TTL-Serial, U1 ESP-01v090, U2 MCP1700-3302E_TO92

Commit message: Updates to schematic and PCB
Parts:
- removed REF** (x2): MountingHole_2.5mm, MountingHole:MountingHole_2.5mm
- C1: footprint Capacitor_THT:CP_Radial_Tantal_D5.0mm_P2.50mm -> Capacitor_THT:C_Disc_D3.8mm_W2.6mm_P2.50mm
- C2, C3: footprint Capacitor_THT:C_Disc_D5.0mm_W2.5mm_P2.50mm -> Capacitor_THT:C_Disc_D3.8mm_W2.6mm_P2.50mm; moved to B.Cu
- J2: footprint Connector_PinHeader_2.00mm:PinHeader_1x03_P2.00mm_Vertical -> Connector_PinHeader_2.54mm:PinHeader_1x03_P2.54mm_Vertical
- moved C2 2.54 mm to (107.3, 79.4), turned to 270 degrees
- moved C3 2.54 mm to (116.8, 79.4), turned to 270 degrees
- moved J2 2.01 mm to (123.2, 99.1)
Connections:
- C2 pad 1: GND -> +3V3
- C2 pad 2: +3V3 -> GND
- C3 pad 1: GND -> Net-(C3-Pad1)
- C3 pad 2: Net-(C3-Pad2) -> GND
- J1 pad 2: Net-(C3-Pad2) -> Net-(C3-Pad1)
- U2 pad 2: Net-(C3-Pad2) -> Net-(C3-Pad1)
Routing:
- net Net-(C3-Pad1): track 0.00 -> 11.5 mm
- net Net-(C3-Pad2): track 11.5 -> 0.00 mm
- net Net-(J2-Pad2): track 6.70 -> 5.50 mm
Other:
- board text added: "+"
- board text added: "G Tx Rx"
